Commit message: Add SO101 task and automatic robot visualization for live and replay

File: packages/robotics/test/warehouse.urdf (robot description, URDF)
Before this commit: robot warehouse, 6 links, 5 joints
Links:
- link base_link: geometry collision box size=0.82 0.66 0.22; visual mesh filename=embedded-stl
- link left_wheel: geometry collision cylinder length=0.13 radius=0.22; visual mesh filename=embedded-stl
- link right_wheel: geometry collision cylinder length=0.13 radius=0.22; visual mesh filename=embedded-stl
